File: Hardware/Segment_Display_Board/Segment_Display_Board.kicad_pcb (KiCad board)
At the start: 2 copper layers, 58.4 x 141 mm, 94 parts, among them J101 IN, J102 OUT, J201 Tag Connect, J202 EXT BTN, J301 USB_B_Micro, J302 PROG, J401 19V Input, Q1001 MMBT3904, Q1002 MMBT3906, Q1101 MMBT3904, Q1102 MMBT3906, Q1201 MMBT3904, Q1202 MMBT3906, Q601 MMBT3904, Q602 MMBT3906, Q701 MMBT3904, Q702 MMBT3906, Q801 MMBT3904, Q802 MMBT3906, Q901 MMBT3904, Q902 MMBT3906, SW201 RESET, SW202 DAY_RESET, SW203 DAY_ADV, SW204 DAY_SUB, U201 ATmega328P-A, U202 DS1307Z+, U301 FT232RL, U401 NCV1117ST50T3G, U501 5inSegment, U502 SN74HC595, Y201 16mHz, Y202 32.768kHz

Commit message: Bump
Parts:
- added TP501: DP, TestPoint:TestPoint_Pad_D1.5mm, F.Cu at (166.2, 139.2)
- R1003, R1103, R1203, R603, R703, R803, R903: value 680R -> TBD
Connections:
- U502 pad 7: unconnected-(U502-Pad7) -> Net-(U502-Pad7)
Routing:
- net Net-(U502-Pad7): track 0.00 -> 4.32 mm
Changed lines of the file:
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@@
   (net 52 "Net-(Q1102-Pad3)")
   (net 53 "unconnected-(U501-Pad6)")
-  (net 54 "unconnected-(U502-Pad7)")
+  (net 54 "Net-(U502-Pad7)")
   (net 55 "/MCU/SDA")
   (net 56 "Net-(U202-Pad1)")
@@
       (effects (font (size 0.75 0.75) (thickness 0.15)))
     )
-    (fp_text value "680R" (at 0 2.5) (layer "F.Fab")
+    (fp_text value "TBD" (at 0 2.5) (layer "F.Fab")
       (effects (font (size 1 1) (thickness 0.15)))
     )
@@
     )
   )
+  (footprint "TestPoint:TestPoint_Pad_D1.5mm" (layer "F.Cu")
+    (at 166.25 139.25)
+    (descr "SMD pad as test Point, diameter 1.5mm")
+    (tags "test point SMD pad")
+    (property "Sheetfile" "display_card.kicad_sch")
+    (property "Sheetname" "Display Card")
+    (attr exclude_from_pos_files)
+    (fp_text reference "TP501" (at 0 -1.648) (layer "F.SilkS") hide
+      (effects (font (size 1 1) (thickness 0.15)))
+    )
+    (fp_text value "DP" (at 0 2) (layer "F.SilkS")
+      (effects (font (size 1 1) (thickness 0.15)))
+    )
+    (fp_text user "${REFERENCE}" (at 0 -1.65) (layer "F.Fab") hide
+      (effects (font (size 1 1) (thickness 0.15)))
+    )
+    (fp_circle (center 0 0) (end 0 0.95) (layer "F.SilkS") (width 0.12) (fill none))
+    (fp_circle (center 0 0) (end 1.25 0) (layer "F.CrtYd") (width 0.05) (fill none))
+    (pad "1" smd circle (at 0 0) (size 1.5 1.5) (layers "F.Cu" "F.Mask")
+      (net 54 "Net-(U502-Pad7)") (pinfunction "1") (pintype "passive"))
+  )
   (footprint "Resistor_SMD:R_0805_2012Metric" (layer "F.Cu")
     (at 159.4125 111.4875 180)
@@
       (effects (font (size 0.75 0.75) (thickness 0.15)))
     )
-    (fp_text value "680R" (at 0 2.5) (layer "F.Fab")
+    (fp_text value "TBD" (at 0 2.5) (layer "F.Fab")
       (effects (font (size 1 1) (thickness 0.15)))
     )
@@
       (effects (font (size 0.75 0.75) (thickness 0.15)))
     )
-    (fp_text value "680R" (at 0 2.5) (layer "F.Fab")
+    (fp_text value "TBD" (at 0 2.5) (layer "F.Fab")
       (effects (font (size 1 1) (thickness 0.15)))
     )
@@
       (effects (font (size 0.75 0.75) (thickness 0.15)))
     )
-    (fp_text value "680R" (at 0 2.5) (layer "F.Fab")
+    (fp_text value "TBD" (at 0 2.5) (layer "F.Fab")
       (effects (font (size 1 1) (thickness 0.15)))
     )
@@
       (effects (font (size 0.75 0.75) (thickness 0.15)))
     )
-    (fp_text value "680R" (at 0 2.5) (layer "F.Fab")
+    (fp_text value "TBD" (at 0 2.5) (layer "F.Fab")
       (effects (font (size 1 1) (thickness 0.15)))
     )
@@
       (effects (font (size 0.75 0.75) (thickness 0.15)))
     )
-    (fp_text value "680R" (at 0 2.5) (layer "F.Fab")
+    (fp_text value "TBD" (at 0 2.5) (layer "F.Fab")
       (effects (font (size 1 1) (thickness 0.15)))
     )
@@
       (net 80 "/Display Card/SEG_G") (pinfunction "QG") (pintype "output"))
     (pad "7" smd roundrect (at -3.4125 1.625 90) (size 1.775 0.5) (layers "F.Cu" "F.Paste" "F.Mask") (roundrect_rratio 0.25)
-      (net 54 "unconnected-(U502-Pad7)") (pinfunction "QH") (pintype "output+no_connect"))
+      (net 54 "Net-(U502-Pad7)") (pinfunction "QH") (pintype "output"))
     (pad "8" smd roundrect (at -3.4125 2.275 90) (size 1.775 0.5) (layers "F.Cu" "F.Paste" "F.Mask") (roundrect_rratio 0.25)
       (net 2 "GND") (pinfunction "GND") (pintype "power_in"))
@@
       (effects (font (size 0.75 0.75) (thickness 0.15)))
     )
-    (fp_text value "680R" (at 0 2.5) (layer "F.Fab")
+    (fp_text value "TBD" (at 0 2.5) (layer "F.Fab")
       (effects (font (size 1 1) (thickness 0.15)))
     )
@@
   (segment (start 156.9625 77.4375) (end 156.9625 77.85) (width 0.25) (layer "F.Cu") (net 52))
   (segment (start 157.55 78.4375) (end 157.55 81.375) (width 0.25) (layer "F.Cu") (net 52))
+  (segment (start 164.75 139.25) (end 166.25 139.25) (width 0.25) (layer "F.Cu") (net 54))
+  (segment (start 163.825 138.325) (end 164.75 139.25) (width 0.25) (layer "F.Cu") (net 54))
+  (segment (start 163.825 136.8125) (end 163.825 138.325) (width 0.25) (layer "F.Cu") (net 54))
   (segment (start 133.5 104.5) (end 132 103) (width 0.25) (layer "F.Cu") (net 55))
   (segment (start 140.981396 50.905) (end 143.225 50.905) (width 0.25) (layer "F.Cu") (net 55))
