File: Hardware/Segment_Display_Board/display_card.kicad_sch (KiCad schematic)
At the start: 5 parts, among them U501 5inSegment, U502 SN74HC595

Commit message: Bump
Parts:
- added TP501: DP, TestPoint:TestPoint_Pad_D1.5mm, symbol Connector:TestPoint
Connections:
- net at U502.7 (QH): now also TP501.1
- no-connect marks 2 -> 1
Changed lines of the file:
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@@
   )
   (no_connect (at 40.005 104.775))
-  (no_connect (at 111.76 108.585))
   (wire (pts (xy 26.035 86.995) (xy 40.005 86.995))
     (stroke (width 0) (type default) (color 0 0 0 0))
@@
     (stroke (width 0) (type default) (color 0 0 0 0))
   )
+  (wire (pts (xy 111.76 108.585) (xy 128.905 108.585))
+    (stroke (width 0) (type default) (color 0 0 0 0))
+  )
   (wire (pts (xy 48.895 114.3) (xy 48.895 113.665))
     (stroke (width 0) (type default) (color 0 0 0 0))
@@
   )
   (wire (pts (xy 88.9 100.965) (xy 93.98 100.965))
+    (stroke (width 0) (type default) (color 0 0 0 0))
+  )
+  (wire (pts (xy 128.905 108.585) (xy 128.905 104.775))
     (stroke (width 0) (type default) (color 0 0 0 0))
   )
@@
       (effects (font (size 1.27 1.27)) hide)
     )
+    (pin "1")
+  )
+  (symbol (lib_id "Connector:TestPoint") (at 128.905 104.775 0) (unit 1)
+    (in_bom yes) (on_board yes)
+    (property "Reference" "TP501" (id 0) (at 130.81 101.6 0)
+      (effects (font (size 1.27 1.27)) (justify left))
+    )
+    (property "Value" "DP" (id 1) (at 130.81 104.14 0)
+      (effects (font (size 1.27 1.27)) (justify left))
+    )
+    (property "Footprint" "TestPoint:TestPoint_Pad_D1.5mm" (id 2) (at 133.985 104.775 0)
+      (effects (font (size 1.27 1.27)) hide)
+    )
+    (property "Datasheet" "~" (id 3) (at 133.985 104.775 0)
+      (effects (font (size 1.27 1.27)) hide)
+    )
